File: fc660a_plate/fc660a_plate.kicad_pcb (KiCad board)
At the start: 2 copper layers, 318.5 x 102.1 mm, 13 parts

Commit message: 3/14/21
Parts:
- removed ? (x10): 660_z_outline, Keyboard_Footprints:660_z_outline
- removed ?: 660_x_outline, Keyboard_Footprints:660_x_outline
- added Plate_Cutout_Alps: , Keyboard_Footprints:Plate_Cutout_Alps, F.Cu at (38.1, 38.1)
- added Plate_Cutout_Alps: , Keyboard_Footprints:Plate_Cutout_Alps, F.Cu at (276.2, 57.1)
- added Plate_Cutout_Alps: , Keyboard_Footprints:Plate_Cutout_Alps, F.Cu at (252.4, 95.2)
- added Plate_Cutout_Alps: , Keyboard_Footprints:Plate_Cutout_Alps, F.Cu at (333.4, 38.1)
- added Plate_Cutout_Alps: , Keyboard_Footprints:Plate_Cutout_Alps, F.Cu at (300.0, 57.1)
- added Plate_Cutout_Alps: , Keyboard_Footprints:Perferation, F.Cu at (77.7, 27.9)
- added Plate_Cutout_Alps: , Keyboard_Footprints:Perferation, F.Cu at (293.8, 27.9)
- added Plate_Cutout_Alps: , Keyboard_Footprints:Perferation, F.Cu at (293.8, 124.5)
- added Plate_Cutout_Alps: , Keyboard_Footprints:Perferation, F.Cu at (77.7, 124.5)
- added Plate_Cutout_Alps: , Keyboard_Footprints:Plate_Cutout_Alps, F.Cu at (283.4, 95.2)
- added Plate_Cutout_Alps: , Keyboard_Footprints:Plate_Cutout_Alps, F.Cu at (292.9, 38.1)
- added Plate_Cutout_Alps: , Keyboard_Footprints:Plate_Cutout_Alps, F.Cu at (57.1, 38.1)
- added Plate_Cutout_Alps: , Keyboard_Footprints:Plate_Cutout_Alps, F.Cu at (195.3, 95.2)
- added Plate_Cutout_Alps: , Keyboard_Footprints:Plate_Cutout_Alps, F.Cu at (50.0, 95.2)
- added Plate_Cutout_Alps: , Keyboard_Footprints:Plate_Cutout_Alps, F.Cu at (261.9, 76.2)
- added Plate_Cutout_Alps: , Keyboard_Footprints:Plate_Cutout_Alps, F.Cu at (190.5, 38.1)
- added Plate_Cutout_Alps: , Keyboard_Footprints:Plate_Cutout_Alps, F.Cu at (226.2, 114.3)
- added Plate_Cutout_Alps: , Keyboard_Footprints:Plate_Cutout_Alps, F.Cu at (133.3, 38.1)
- added Plate_Cutout_Alps: , Keyboard_Footprints:Plate_Cutout_Alps, F.Cu at (138.1, 95.2)
- added Plate_Cutout_Alps: , Keyboard_Footprints:Plate_Cutout_Alps, F.Cu at (100.0, 95.2)
- added Plate_Cutout_Alps: , Keyboard_Footprints:Plate_Cutout_Alps, F.Cu at (109.5, 76.2)
- added Plate_Cutout_Alps: , Keyboard_Footprints:Plate_Cutout_Alps, F.Cu at (181.0, 57.1)
- added Plate_Cutout_Alps: , Keyboard_Footprints:Plate_Cutout_Alps, F.Cu at (76.2, 38.1)
- added Plate_Cutout_Alps: , Keyboard_Footprints:Plate_Cutout_Alps, F.Cu at (273.8, 114.3)
- added Plate_Cutout_Alps: , Keyboard_Footprints:Plate_Cutout_Alps, F.Cu at (147.6, 76.2)
- added Plate_Cutout_Alps: , Keyboard_Footprints:Plate_Cutout_Alps, F.Cu at (185.7, 76.2)
- added Plate_Cutout_Alps: , Keyboard_Footprints:Plate_Cutout_Alps, F.Cu at (257.2, 57.1)
- added Plate_Cutout_Alps: , Keyboard_Footprints:Plate_Cutout_Alps, F.Cu at (242.9, 76.2)
- added Plate_Cutout_Alps: , Keyboard_Footprints:Plate_Cutout_Alps, F.Cu at (200.0, 57.1)
- added Plate_Cutout_Alps: , Keyboard_Footprints:Plate_Cutout_Alps, F.Cu at (238.1, 57.1)
- added Plate_Cutout_Alps: , Keyboard_Footprints:Plate_Cutout_Alps, F.Cu at (250.0, 114.3)
- added Plate_Cutout_Alps: , Keyboard_Footprints:Plate_Cutout_Alps, F.Cu at (292.9, 76.2)
- added Plate_Cutout_Alps: , Keyboard_Footprints:Plate_Cutout_Alps, F.Cu at (66.7, 57.1)
- added Plate_Cutout_Alps: , Keyboard_Footprints:Plate_Cutout_Alps, F.Cu at (95.2, 38.1)
- added Plate_Cutout_Alps: , Keyboard_Footprints:Plate_Cutout_Alps, F.Cu at (228.6, 38.1)
- added Plate_Cutout_Alps: , Keyboard_Footprints:Plate_Cutout_Alps, F.Cu at (71.4, 76.2)
- added Plate_Cutout_Alps: , Keyboard_Footprints:Plate_Cutout_Alps, F.Cu at (223.8, 76.2)
- added Plate_Cutout_Alps: , Keyboard_Footprints:Plate_Cutout_Alps, F.Cu at (123.8, 57.1)
- added Plate_Cutout_Alps: , Keyboard_Footprints:Plate_Cutout_Alps, F.Cu at (81.0, 95.2)
- added Plate_Cutout_Alps: , Keyboard_Footprints:Plate_Cutout_Alps, F.Cu at (219.1, 57.1)
- added Plate_Cutout_Alps: , Keyboard_Footprints:Plate_Cutout_Alps, F.Cu at (247.7, 38.1)
- added Plate_Cutout_Alps: , Keyboard_Footprints:Plate_Cutout_Alps, F.Cu at (161.9, 57.1)
- added Plate_Cutout_Alps: , Keyboard_Footprints:Plate_Cutout_Alps, F.Cu at (152.4, 38.1)
- added Plate_Cutout_Alps: , Keyboard_Footprints:Plate_Cutout_Alps, F.Cu at (171.4, 38.1)
- added Plate_Cutout_Alps: , Keyboard_Footprints:Plate_Cutout_Alps, F.Cu at (114.3, 38.1)
- added Plate_Cutout_Alps: , Keyboard_Footprints:Plate_Cutout_Alps, F.Cu at (85.7, 57.1)
- added Plate_Cutout_Alps: , Keyboard_Footprints:Plate_Cutout_Alps, F.Cu at (40.5, 114.3)
- added Plate_Cutout_Alps: , Keyboard_Footprints:Plate_Cutout_Alps, F.Cu at (214.3, 95.2)
- added Plate_Cutout_Alps: , Keyboard_Footprints:Plate_Cutout_Alps, F.Cu at (176.2, 95.2)
- added Plate_Cutout_Alps: , Keyboard_Footprints:Plate_Cutout_Alps, F.Cu at (333.4, 114.3)
- added Plate_Cutout_Alps: , Keyboard_Footprints:Plate_Cutout_Alps, F.Cu at (314.3, 95.2)
- added Plate_Cutout_Alps: , Keyboard_Footprints:Plate_Cutout_Alps, F.Cu at (157.2, 95.2)
- added Plate_Cutout_Alps: , Keyboard_Footprints:Plate_Cutout_Alps, F.Cu at (90.5, 76.2)
- added Plate_Cutout_Alps: , Keyboard_Footprints:Plate_Cutout_Alps, F.Cu at (42.9, 57.1)
- added Plate_Cutout_Alps: , Keyboard_Footprints:Plate_Cutout_Alps, F.Cu at (233.4, 95.2)
- added Plate_Cutout_Alps: , Keyboard_Footprints:Plate_Cutout_Alps, F.Cu at (333.4, 57.1)
- added Plate_Cutout_Alps: , Keyboard_Footprints:Plate_Cutout_Alps, F.Cu at (142.9, 57.1)
- added Plate_Cutout_Alps: , Keyboard_Footprints:Plate_Cutout_Alps, F.Cu at (209.6, 38.1)
- added Plate_Cutout_Alps: , Keyboard_Footprints:Plate_Cutout_Alps, F.Cu at (166.7, 76.2)
- added Plate_Cutout_Alps: , Keyboard_Footprints:Plate_Cutout_Alps, F.Cu at (119.1, 95.2)
- added Plate_Cutout_Alps: , Keyboard_Footprints:Plate_Cutout_Alps, F.Cu at (104.8, 57.1)
- added Plate_Cutout_Alps: , Keyboard_Footprints:Plate_Cutout_Alps, F.Cu at (204.8, 76.2)
- added Plate_Cutout_Alps: , Keyboard_Footprints:Plate_Cutout_Alps, F.Cu at (128.6, 76.2)
- added Plate_Cutout_Alps: , Keyboard_Footprints:Plate_Cutout_Alps, F.Cu at (266.7, 38.1)
- added Plate_Cutout_Alps: , Keyboard_Footprints:Plate_Cutout_Alps, F.Cu at (314.3, 114.3)
- added Plate_Cutout_Alps: , Keyboard_Footprints:Plate_Cutout_Alps, F.Cu at (295.3, 114.3)
- added Plate_Cutout_Alps_2: , Keyboard_Footprints:Plate_Cutout_Alps_2, F.Cu at (88.1, 114.3)
- added Plate_Cutout_Alps_2: , Keyboard_Footprints:Plate_Cutout_Alps_2, F.Cu at (45.2, 76.2)
- added Plate_Cutout_Alps_2: , Keyboard_Footprints:Plate_Cutout_Alps_2, F.Cu at (83.3, 114.3)
- added Plate_Cutout_Alps_2: , Keyboard_Footprints:Plate_Cutout_Alps_2, F.Cu at (166.7, 114.3)
- added Plate_Cutout_Alps_2: , Keyboard_Footprints:Plate_Cutout_Alps_2, F.Cu at (64.3, 114.3)
- added Plate_Cutout_Alps_2: , Keyboard_Footprints:Plate_Cutout_Alps_2, F.Cu at (61.9, 114.3)
- added Plate_Cutout_Alps_2: , Keyboard_Footprints:Plate_Cutout_Alps_2, F.Cu at (154.8, 114.3)
- added Plate_Cutout_Alps_2: , Keyboard_Footprints:Plate_Cutout_Alps_2, F.Cu at (40.5, 76.2)
- added Screw_Hole: , Keyboard_Footprints:Screw_Hole, F.Cu at (52.4, 114.3)
- added Screw_Hole: , Keyboard_Footprints:Screw_Hole, F.Cu at (323.9, 114.3)
- added Screw_Hole: , Keyboard_Footprints:Screw_Hole, F.Cu at (157.2, 76.2)
- added Screw_Hole: , Keyboard_Footprints:Screw_Hole, F.Cu at (247.7, 57.1)
- Screw_Hole: renamed from screw_hole; footprint Keyboard_Footprints:screw_hole -> Keyboard_Footprints:FC660m_small_hole
- Screw_Hole: renamed from screw_hole; footprint Keyboard_Footprints:screw_hole -> Keyboard_Footprints:Screw_Hole
Other:
- board size 318.5 x 102.1 mm -> 318.5 x 106.6 mm
- net class Default removed
- rule pad_to_mask_clearance: 0.2 -> 0
