File: alps66.kicad_pcb (KiCad board)
At the start: 2 copper layers, 313.3 x 94.7 mm, 188 parts, among them J1 USB_mini_micro_B, K00 KEYSW, K00_1 KEYSW, K01 KEYSW, K02 KEYSW, K03 KEYSW, K04 KEYSW, K05 KEYSW, K06 KEYSW, K07 KEYSW, K10 KEYSW, K11 KEYSW, K12 KEYSW, K13 KEYSW, K14 KEYSW, K15 KEYSW, K16 KEYSW, K17 KEYSW, K20 KEYSW, K21 KEYSW, K22 KEYSW, K23 KEYSW, K24 KEYSW, K25 KEYSW, K26 KEYSW, K26_1 KEYSW, K27 KEYSW, K30 KEYSW, K30_1 KEYSW, K31 KEYSW, K31_1 KEYSW, K32 KEYSW, K32_1 KEYSW, K32_2 KEYSW, K33 KEYSW, K34 KEYSW, K35 KEYSW, K36 KEYSW, K37 KEYSW, K40 KEYSW, K40_1 KEYSW, K40_2 KEYSW, K41 KEYSW, K42 KEYSW, K43 KEYSW, K44 KEYSW, K45 KEYSW, K46 KEYSW, K47 KEYSW, K50 KEYSW, K50_1 KEYSW, K50_2 KEYSW, K51 KEYSW, K52 KEYSW, K53 KEYSW, K54 KEYSW, K55 KEYSW, K56 KEYSW, K57 KEYSW, K60 KEYSW, K60_1 KEYSW, K60_2 KEYSW, K61 KEYSW, K62 KEYSW, K63 KEYSW, K64 KEYSW, K65 KEYSW, K66 KEYSW, K67 KEYSW, K70 KEYSW, K70_1 KEYSW, K71 KEYSW, K72 KEYSW, K73 KEYSW, K74 KEYSW, K75 KEYSW, K76 KEYSW, K77 KEYSW, K80 KEYSW, K81 KEYSW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

Commit message: 3/14/21
Parts:
- removed the 6u_stab at (157.2, 114.3)
- removed the ? at (333.5, 80.5)
- removed D00, D01, D02, D03, D04, D05, D06, D07, D41, D80, D81, D90, D91: D, keyboard_parts:D_SOD123_axial
- removed FC660c_big_hole: , Keyboard_Footprints:FC660c_big_hole
- removed FC660c_small_hole (x2): , Keyboard_Footprints:FC660c_small_hole
- removed K00, K01, K02, K03, K04, K05, K06, K07, K41, K80, K81, K90, K91: KEYSW, Keyboard_Footprints:Alps_SKCM_Reversed
- removed K26_1, K31_1: KEYSW, Keyboard_Footprints:Alps_SKCM_Reversed_Secondary
- removed LED1: LED, keyboard_parts:LED_2012_HSOL
- removed P1: GND, keyboard_parts:PIN_1
- removed P2: 5V, keyboard_parts:PIN_1
- removed SJ1, SJ2: SOLDER_JUMPER, keyboard_parts:SOLDER_JUMPER_2
- removed Via (x2): Via, Keyboard_Footprints:Via
- added ?: , Keyboard_Footprints:TMK_Logo, B.Cu at (330.0, 80.5)
- added D0: D, Keyboard_Footprints:Diode_123_Axial, B.Cu at (261.5, 104.0)
- added D1: D, Keyboard_Footprints:Diode_123_Axial, B.Cu at (204.8, 95.2)
- added D18: D, Keyboard_Footprints:Diode_123_Axial, B.Cu at (338.5, 95.2)
- added D2: D, Keyboard_Footprints:Diode_123_Axial, B.Cu at (223.8, 95.2)
- added D28: D, Keyboard_Footprints:Diode_123_Axial, B.Cu at (333.8, 95.2)
- added D3: D, Keyboard_Footprints:Diode_123_Axial, B.Cu at (214.3, 76.2)
- added D4: D, Keyboard_Footprints:Diode_123_Axial, B.Cu at (220.8, 65.5)
- added D5: D, Keyboard_Footprints:Diode_123_Axial, B.Cu at (228.6, 57.1)
- added D6: D, Keyboard_Footprints:Diode_123_Axial, B.Cu at (238.1, 38.1)
- added D7: D, Keyboard_Footprints:Diode_123_Axial, B.Cu at (257.2, 38.1)
- added D78: D, Keyboard_Footprints:Diode_123_Axial, B.Cu at (216.8, 104.0)
- added D8: D, Keyboard_Footprints:Diode_123_Axial, B.Cu at (334.8, 46.0)
- added K0: KEYSW, Keyboard_Footprints:Alps, F.Cu at (271.5, 114.3)
- added K1: KEYSW, Keyboard_Footprints:Alps, F.Cu at (195.3, 95.2)
- added K18: KEYSW, Keyboard_Footprints:Alps, F.Cu at (333.4, 57.1)
- added K2: KEYSW, Keyboard_Footprints:Alps, F.Cu at (214.3, 95.2)
- added K27_1: KEYSW, Keyboard_Footprints:Alps_Secondary, F.Cu at (295.3, 38.1)
- added K28: KEYSW, Keyboard_Footprints:Alps, F.Cu at (333.4, 114.3)
- added K3: KEYSW, Keyboard_Footprints:Alps, F.Cu at (204.8, 76.2)
- added K4: KEYSW, Keyboard_Footprints:Alps, F.Cu at (223.8, 76.2)
- added K40_3: KEYSW, Keyboard_Footprints:Alps_Secondary, F.Cu at (69.1, 114.3)
- added K5: KEYSW, Keyboard_Footprints:Alps, F.Cu at (219.1, 57.1)
- added K50_3: KEYSW, Keyboard_Footprints:Alps_Secondary, F.Cu at (95.2, 114.3)
- added K6: KEYSW, Keyboard_Footprints:Alps, F.Cu at (228.6, 38.1)
- added K7: KEYSW, Keyboard_Footprints:Alps, F.Cu at (247.7, 38.1)
- added K70_2: KEYSW, Keyboard_Footprints:Alps_Secondary_Reversed, F.Cu at (245.3, 114.3)
- added K78: KEYSW, Keyboard_Footprints:Alps, F.Cu at (219.1, 114.3)
- added K78_1: KEYSW, Keyboard_Footprints:Alps_Secondary_Reversed, F.Cu at (226.2, 114.3)
- added K8: KEYSW, Keyboard_Footprints:Alps, F.Cu at (333.4, 38.1)
- added LED1_0: 3mm, LED_THT:LED_D3.0mm, F.Cu at (57.0, 76.2)
- added LED1_1: 5mm_Rectangular, LED_THT:LED_Rectangular_W5.0mm_H2.0mm, F.Cu at (36.8, 43.2)
- added Pin1: 5V, Keyboard_Footprints:Pin, F.Cu at (124.5, 102.8)
- added Pin2: GND, Keyboard_Footprints:Pin, F.Cu at (128.5, 102.8)
- added Pin3: PC4, Keyboard_Footprints:Pin, F.Cu at (132.5, 102.8)
- added R5: 10k, Resistor_SMD:R_0805_2012Metric, B.Cu at (333.8, 70.0)
- C1: footprint Capacitors_SMD:C_1206 -> Capacitor_SMD:C_0805_2012Metric
- C2, C3, C4, C5, C6: footprint Capacitors_SMD:C_0805 -> Capacitor_SMD:C_0805_2012Metric
- D10, D11, D12, D13, D14, D15, D16, D17, D20, D21, D22, D23, D24, D25, D26, D27, D30, D31, D32, D33, D34, D35, D36, D37, D40, D42, D43, D44, D45, D46, D47, D50, D51, D52, D53, D54, D55, D56, D57, D60, D61, D62, D63, D64, D65, D66, D67, D70, D71, D72, D73, D74, D75, D76, D77: footprint keyboard_parts:D_SOD123_axial -> Keyboard_Footprints:Diode_123_Axial
- J1: footprint keyboard_parts:USB_miniB_hirose_5S8 -> Keyboard_Footprints:USB_miniB_hirose_5S8
- K00_1, K30_1, K32_1, K32_2, K40_1, K40_2, K70_1: footprint Keyboard_Footprints:Alps_SKCM_Reversed_Secondary -> Keyboard_Footprints:Alps_Secondary
- K10, K11, K12, K13, K14, K15, K16, K17, K20, K21, K22, K23, K24, K25, K26, K27, K30, K31, K32, K33, K34, K35, K36, K37, K40, K42, K43, K44, K45, K46, K47, K51, K52, K53, K54, K55, K56, K57, K61, K62, K63, K64, K65, K66, K67, K70, K71, K72, K73, K74, K75, K76, K77: footprint Keyboard_Footprints:Alps_SKCM_Reversed -> Keyboard_Footprints:Alps
- K50, K60: footprint Keyboard_Footprints:Alps_SKCM -> Keyboard_Footprints:Alps
- K50_1, K50_2, K60_1, K60_2: footprint Keyboard_Footprints:Alps_SKCM_Reversed_Secondary -> Keyboard_Footprints:Alps_Secondary_Reversed
- Oval_Mounting_Hole (x7): renamed from Poker_oval_hole; footprint Keyboard_Footprints:Poker_oval_hole -> Keyboard_Footprints:Oval_Mounting_Hole
- R1, R2: footprint Resistors_SMD:R_0805 -> Resistor_SMD:R_0805_2012Metric
- R3, R4: value 1K -> 1k; footprint Resistors_SMD:R_0805 -> Resistor_SMD:R_0805_2012Metric
- SW1: renamed from SW100; footprint Buttons_Switches_SMD:SW_SPST_B3U-1000P-B -> Button_Switch_SMD:SW_SPST_B3U-1000P-B
- U1: footprint keyboard_parts:QFP32_reflow -> Package_QFP:LQFP-32_7x7mm_P0.8mm
- X1: value CRYSTAL -> 16MHz_12pF; footprint keyboard_parts:FA-238 -> Crystal:Crystal_SMD_SeikoEpson_FA238-4Pin_3.2x2.5mm
- moved D70 36.1 mm to (243.0, 104.0), turned to 180 degrees
- moved R2 31.8 mm to (170.8, 105.5), turned to 180 degrees
- moved R1 30.7 mm to (170.8, 102.8), turned to 180 degrees
- moved K27 28.6 mm to (304.8, 38.1), turned to 180 degrees
- moved D27 27.1 mm to (311.8, 57.1), turned to -90 degrees
- moved D40 22.2 mm to (68.2, 106.2), turned to 180 degrees
- moved C1 20.7 mm to (142.5, 109.8)
- moved D63 18.8 mm to (154.5, 65.5), turned to 180 degrees
- moved D25 15.5 mm to (274.0, 46.0), turned to 180 degrees
- moved D31 15.3 mm to (40.5, 95.2), turned to -90 degrees
- moved D22 11.4 mm to (324.2, 95.2), turned to -90 degrees
- moved D30 11.3 mm to (33.0, 95.2), turned to -90 degrees
- moved D34 10.5 mm to (33.3, 57.1), turned to -90 degrees
- moved K31 9.52 mm to (50.0, 95.2)
- moved R4 8.84 mm to (59.0, 79.5)
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Connections:
- J1 pad 4: Net-(J1-Pad4) -> unconnected-(J1-Pad4)
- J1 pad 6: Net-(J1-Pad6) -> unconnected-(J1-Pad6)
- U1 pad 22: Net-(K80-Pad1) -> /col8
- U1 pad 23: Net-(K81-Pad1) -> unconnected-(U1-Pad23)
- X1 pad 2: Net-(C3-Pad1) -> GND
- X1 pad 3: GND -> Net-(C3-Pad1)
Routing:
- net /col8: track 0.00 -> 452.9 mm, vias 0 -> 1
- net Net-(K81-Pad1): track 376.9 -> 0.00 mm, vias 2 -> 0
- net Net-(D90-Pad1): track 338.6 -> 0.00 mm, vias 2 -> 0
- net Net-(K80-Pad1): track 292.1 -> 0.00 mm, vias 1 -> 0
- net Net-(Pin3-Pad1): track 240.9 -> 7.77 mm, vias 1 -> 0
- net GND: track 535.2 -> 366.9 mm, vias 30 -> 8
- net Net-(D91-Pad2): track 108.6 -> 0.00 mm
- net /row0: track 231.6 -> 322.7 mm
- net /row1: track 298.9 -> 375.1 mm
- net Net-(R5-Pad1): track 312.1 -> 236.0 mm, vias 4 -> 2
- net Net-(LED1_0-Pad1): track 3.25 -> 54.9 mm, vias 0 -> 1
- net Net-(D80-Pad2): track 47.7 -> 0.00 mm
- net Net-(D0-Pad2): track 69.4 -> 25.4 mm
- net +5V: track 281.2 -> 324.7 mm, vias 1 -> 5
- net Net-(D18-Pad2): track 0.00 -> 39.8 mm
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- removed copper zone on F.Cu, net GND
Other:
- outline, holes or cut-outs redrawn
- net class 20mil removed
- net class 6mil removed
- net class 8mil removed
- net class Default removed
- net class Power removed
- rule pad_to_mask_clearance: 0.2 -> 0
- board text added: "Alps66 Rev 2.0 Based on a Hasu Design"
- board text removed: "Alps66 Rev 1.1 By Andrew D Based on a Hasu Design"

Commit message: Update Axial_Diode Footprint
Parts:
- turned D0 to 0 degrees
- turned D1 to 90 degrees
- turned D10 to 90 degrees
- turned D11 to 90 degrees
- turned D12 to 90 degrees
- turned D13 to 90 degrees
- turned D14 to 90 degrees
- turned D15 to 0 degrees
- turned D16 to 90 degrees
- turned D17 to 90 degrees
- turned D18 to 90 degrees
- turned D2 to 90 degrees
- turned D20 to 90 degrees
- turned D21 to 90 degrees
- turned D22 to 90 degrees
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